File: Boost converter.brd (EAGLE design)
At the start: 25.1 x 63.5 mm, 21 parts, among them IC1 NE555N, IC2 attiny84, IC3 attiny85, Q1 2n7000, Q2 zvp4105

Commit message: Rerouted USB data lines
rerouted usb D- line to pin 6 on the attiny84 socket and D+ line to pin 5(int0) on attiny84 socket. pins 2 and 3 on socket were left unconnected but I still need to add crystal oscillator to board and connect it to these pins
Connections:
- net N$4: now also IC2.6; no longer IC2.2
- net N$5: now also IC2.5; no longer IC2.3
Routing:
- net N$4: track 21.5 -> 12.0 mm
- net N$5: track 17.9 -> 12.8 mm
Changed lines of the file:
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@@
 <wire x1="12.6492" y1="7.62" x2="12.7" y2="7.62" width="0.1524" layer="1"/>
-</signal>
-<signal name="N$4">
-<contactref element="IC2" pad="2"/>
-<contactref element="R5" pad="2"/>
-<wire x1="3.81" y1="32.3088" x2="3.81" y2="33.02" width="0.1524" layer="1"/>
-<wire x1="9.906" y1="26.2128" x2="3.81" y2="32.3088" width="0.1524" layer="1"/>
-<wire x1="9.906" y1="17.9832" x2="9.906" y2="26.2128" width="0.1524" layer="1"/>
-<wire x1="12.6492" y1="15.24" x2="9.906" y2="17.9832" width="0.1524" layer="1"/>
-<wire x1="12.6492" y1="15.24" x2="12.7" y2="15.24" width="0.1524" layer="1"/>
-</signal>
-<signal name="N$5">
-<contactref element="IC2" pad="3"/>
-<contactref element="R6" pad="2"/>
-<wire x1="3.81" y1="29.8704" x2="3.81" y2="30.48" width="0.1524" layer="16"/>
-<wire x1="9.906" y1="23.7744" x2="3.81" y2="29.8704" width="0.1524" layer="16"/>
-<wire x1="9.906" y1="15.3924" x2="9.906" y2="23.7744" width="0.1524" layer="16"/>
-<wire x1="10.0584" y1="15.24" x2="9.906" y2="15.3924" width="0.1524" layer="16"/>
-<wire x1="10.0584" y1="15.24" x2="10.16" y2="15.24" width="0.1524" layer="16"/>
 </signal>
 <signal name="N$1">
@@
 <wire x1="7.62" y1="43.2816" x2="7.62" y2="43.18" width="0.1524" layer="1"/>
 </signal>
+<signal name="N$4">
+<contactref element="R5" pad="2"/>
+<contactref element="IC2" pad="6"/>
+<wire x1="11.43" y1="15.24" x2="12.7" y2="15.24" width="0.1524" layer="16"/>
+<wire x1="3.81" y1="22.86" x2="11.43" y2="15.24" width="0.1524" layer="16"/>
+</signal>
+<signal name="N$5">
+<contactref element="R6" pad="2"/>
+<contactref element="IC2" pad="5"/>
+<wire x1="3.81" y1="24.6888" x2="3.81" y2="25.4" width="0.1524" layer="1"/>
+<wire x1="10.0584" y1="18.4404" x2="3.81" y2="24.6888" width="0.1524" layer="1"/>
+<wire x1="10.0584" y1="15.24" x2="10.0584" y2="18.4404" width="0.1524" layer="1"/>
+<wire x1="10.0584" y1="15.24" x2="10.16" y2="15.24" width="0.1524" layer="1"/>
+</signal>
 </signals>

Commit message: Added crystal oscillator
also had to move around boost converter components to make room for the oscillator, not sure how drastic the inductance and capacitance changes from the pcb lines will be and if it will have a large impact on boost converter output voltage. if I do get this new board fabricated and the voltage does change significantly, I can just switch out the converter diode to drop the voltage to the right level. also added line from attiny84 io pin to attiny85 pb3 on pin 2
Parts:
- added Q3: (no value), special:QS
- moved C1 5.08 mm to (3.81, 53.3)
- moved Q1 4.58 mm to (11.4, 41.9)
- moved D1 2.84 mm to (6.35, 47.0)
- moved R1 2.54 mm to (1.27, 55.9)
Connections:
- new net N$11: IC2.13, IC3.2
- new net N$16: IC2.3, Q3.1
- new net N$17: IC2.2, Q3.2
Routing:
- net N$11: track 0.00 -> 15.7 mm
- net N$17: track 0.00 -> 14.4 mm
- net N$16: track 0.00 -> 10.9 mm
- net N$14: track 6.31 -> 2.46 mm
- net N$15: track 18.5 -> 22.2 mm
- net V+: track 47.1 -> 45.6 mm
- net VCC: track 66.4 -> 65.9 mm
